Commit message: adds xacro parameters to build model with different collision types

File: ur_description/urdf/inc/ur_macro.xacro (robot description, xacro)
@@ -53,5 +53,6 @@
     safety_limits:=false
     safety_pos_margin:=0.15
-    safety_k_position:=20"
+    safety_k_position:=20
+    collision_type:=mesh"
   >
     <!-- Load configuration data from the provided .yaml files -->
@@ -75,10 +76,40 @@
         </material>
       </visual>
-      <collision>
-        <origin xyz="0 0 0" rpy="0 0 ${pi}"/>
-        <geometry>
-          <mesh filename="${base_collision_mesh}"/>
-        </geometry>
-      </collision>
+      <!-- Collision geometry: mesh or primitives based on collision_type -->
+      <xacro:if value="${collision_type == 'mesh'}">
+        <collision>
+          <origin xyz="0 0 0" rpy="0 0 ${pi}"/>
+          <geometry>
+            <mesh filename="${base_collision_mesh}"/>
+          </geometry>
+        </collision>
+      </xacro:if>
+      <xacro:if value="${collision_type == 'cylinder'}">
+        <collision>
+          <origin xyz="0 0 0" rpy="0 0 0"/>
+          <geometry>
+            <cylinder radius="${base_inertia_radius}" length="${base_inertia_length}"/>
+          </geometry>
+        </collision>
+      </xacro:if>
+      <xacro:if value="${collision_type == 'capsule'}">
+        <xacro:capsule_collision radius="${base_inertia_radius}" length="${base_inertia_length}" x="0" y="0" z="0" roll="0" pitch="0" yaw="0"/>
+      </xacro:if>
+      <xacro:if value="${collision_type == 'sphere'}">
+        <collision>
+          <origin xyz="0 0 0" rpy="0 0 0"/>
+          <geometry>
+            <sphere radius="${base_inertia_radius}"/>
+          </geometry>
+        </collision>
+      </xacro:if>
+      <xacro:if value="${collision_type == 'box'}">
+        <collision>
+          <origin xyz="0 0 0" rpy="0 0 0"/>
+          <geometry>
+            <box size="${2*base_inertia_radius} ${2*base_inertia_radius} ${base_inertia_length}"/>
+          </geometry>
+        </collision>
+      </xacro:if>
       <xacro:cylinder_inertial radius="${base_inertia_radius}" length="${base_inertia_length}" mass="${base_mass}">
         <origin xyz="0 0 0" rpy="0 0 0" />
@@ -95,10 +126,40 @@
         </material>
       </visual>
-      <collision>
-        <origin xyz="0 0 0" rpy="0 0 ${pi}"/>
-        <geometry>
-          <mesh filename="${shoulder_collision_mesh}"/>
-        </geometry>
-      </collision>
+      <!-- Collision geometry: mesh or primitives based on collision_type -->
+      <xacro:if value="${collision_type == 'mesh'}">
+        <collision>
+          <origin xyz="0 0 0" rpy="0 0 ${pi}"/>
+          <geometry>
+            <mesh filename="${shoulder_collision_mesh}"/>
+          </geometry>
+        </collision>
+      </xacro:if>
+      <xacro:if value="${collision_type == 'cylinder'}">
+        <collision>
+          <origin xyz="0 0 0" rpy="0 0 0"/>
+          <geometry>
+            <cylinder radius="${shoulder_radius}" length="${shoulder_offset * 2}"/>
+          </geometry>
+        </collision>
+      </xacro:if>
+      <xacro:if value="${collision_type == 'capsule'}">
+        <xacro:capsule_collision radius="${shoulder_radius}" length="${shoulder_offset * 2}" x="0" y="0" z="0" roll="0" pitch="0" yaw="0"/>
+      </xacro:if>
+      <xacro:if value="${collision_type == 'sphere'}">
+        <collision>
+          <origin xyz="0 0 0" rpy="0 0 0"/>
+          <geometry>
+            <sphere radius="${shoulder_radius}"/>
+          </geometry>
+        </collision>
+      </xacro:if>
+      <xacro:if value="${collision_type == 'box'}">
+        <collision>
+          <origin xyz="0 0 0" rpy="0 0 0"/>
+          <geometry>
+            <box size="${2*shoulder_radius} ${2*shoulder_radius} ${shoulder_offset * 2}"/>
+          </geometry>
+        </collision>
+      </xacro:if>
       <inertial>
         <mass value="${shoulder_mass}"/>
@@ -124,10 +185,40 @@
         </material>
       </visual>
-      <collision>
-        <origin xyz="0 0 ${shoulder_offset}" rpy="${pi/2} 0 ${-pi/2}"/>
-        <geometry>
-          <mesh filename="${upper_arm_collision_mesh}"/>
-        </geometry>
-      </collision>
+      <!-- Collision geometry: mesh or primitives based on collision_type -->
+      <xacro:if value="${collision_type == 'mesh'}">
+        <collision>
+          <origin xyz="0 0 ${shoulder_offset}" rpy="${pi/2} 0 ${-pi/2}"/>
+          <geometry>
+            <mesh filename="${upper_arm_collision_mesh}"/>
+          </geometry>
+        </collision>
+      </xacro:if>
+      <xacro:if value="${collision_type == 'cylinder'}">
+        <collision>
+          <origin xyz="${forearm_x/2} 0 ${shoulder_offset}" rpy="0 ${pi/2} 0"/>
+          <geometry>
+            <cylinder radius="${upper_arm_radius}" length="${-forearm_x if forearm_x &lt; 0 else forearm_x}"/>
+          </geometry>
+        </collision>
+      </xacro:if>
+      <xacro:if value="${collision_type == 'capsule'}">
+        <xacro:capsule_collision radius="${upper_arm_radius}" length="${-forearm_x if forearm_x &lt; 0 else forearm_x}" x="${forearm_x/2}" y="0" z="${shoulder_offset}" roll="0" pitch="${pi/2}" yaw="0"/>
+      </xacro:if>
+      <xacro:if value="${collision_type == 'sphere'}">
+        <collision>
+          <origin xyz="${forearm_x/2} 0 ${shoulder_offset}" rpy="0 0 0"/>
+          <geometry>
+            <sphere radius="${upper_arm_radius}"/>
+          </geometry>
+        </collision>
+      </xacro:if>
+      <xacro:if value="${collision_type == 'box'}">
+        <collision>
+          <origin xyz="${forearm_x/2} 0 ${shoulder_offset}" rpy="0 ${pi/2} 0"/>
+          <geometry>
+            <box size="${2*upper_arm_radius} ${2*upper_arm_radius} ${-forearm_x if forearm_x &lt; 0 else forearm_x}"/>
+          </geometry>
+        </collision>
+      </xacro:if>
       <inertial>
         <mass value="${upper_arm_mass}"/>
@@ -153,10 +244,40 @@
         </material>
       </visual>
-      <collision>
-        <origin xyz="0 0 ${elbow_offset}" rpy="${pi/2} 0 ${-pi/2}"/>
-        <geometry>
-          <mesh filename="${forearm_collision_mesh}"/>
-        </geometry>
-      </collision>
+      <!-- Collision geometry: mesh or primitives based on collision_type -->
+      <xacro:if value="${collision_type == 'mesh'}">
+        <collision>
+          <origin xyz="0 0 ${elbow_offset}" rpy="${pi/2} 0 ${-pi/2}"/>
+          <geometry>
+            <mesh filename="${forearm_collision_mesh}"/>
+          </geometry>
+        </collision>
+      </xacro:if>
+      <xacro:if value="${collision_type == 'cylinder'}">
+        <collision>
+          <origin xyz="${wrist_1_x/2} 0 ${elbow_offset}" rpy="0 ${pi/2} 0"/>
+          <geometry>
+            <cylinder radius="${forearm_radius}" length="${-wrist_1_x if wrist_1_x &lt; 0 else wrist_1_x}"/>
+          </geometry>
+        </collision>
+      </xacro:if>
+      <xacro:if value="${collision_type == 'capsule'}">
+        <xacro:capsule_collision radius="${forearm_radius}" length="${-wrist_1_x if wrist_1_x &lt; 0 else wrist_1_x}" x="${wrist_1_x/2}" y="0" z="${elbow_offset}" roll="0" pitch="${pi/2}" yaw="0"/>
+      </xacro:if>
+      <xacro:if value="${collision_type == 'sphere'}">
+        <collision>
+          <origin xyz="${wrist_1_x/2} 0 ${elbow_offset}" rpy="0 0 0"/>
+          <geometry>
+            <sphere radius="${forearm_radius}"/>
+          </geometry>
+        </collision>
+      </xacro:if>
+      <xacro:if value="${collision_type == 'box'}">
+        <collision>
+          <origin xyz="${wrist_1_x/2} 0 ${elbow_offset}" rpy="0 ${pi/2} 0"/>
+          <geometry>
+            <box size="${2*forearm_radius} ${2*forearm_radius} ${-wrist_1_x if wrist_1_x &lt; 0 else wrist_1_x}"/>
+          </geometry>
+        </collision>
+      </xacro:if>
       <inertial>
         <mass value="${forearm_mass}"/>
@@ -183,10 +304,40 @@
         </material>
       </visual>
-      <collision>
-        <origin xyz="0 0 ${wrist_1_visual_offset}" rpy="${pi/2} 0 0"/>
-        <geometry>
-          <mesh filename="${wrist_1_collision_mesh}"/>
-        </geometry>
-      </collision>
+      <!-- Collision geometry: mesh or primitives based on collision_type -->
+      <xacro:if value="${collision_type == 'mesh'}">
+        <collision>
+          <origin xyz="0 0 ${wrist_1_visual_offset}" rpy="${pi/2} 0 0"/>
+          <geometry>
+            <mesh filename="${wrist_1_collision_mesh}"/>
+          </geometry>
+        </collision>
+      </xacro:if>
+      <xacro:if value="${collision_type == 'cylinder'}">
+        <collision>
+          <origin xyz="0 0 ${wrist_1_visual_offset}" rpy="0 0 0"/>
+          <geometry>
+            <cylinder radius="${wrist_radius}" length="${wrist_1_z if wrist_1_z > 0 else -wrist_1_z}"/>
+          </geometry>
+        </collision>
+      </xacro:if>
+      <xacro:if value="${collision_type == 'capsule'}">
+        <xacro:capsule_collision radius="${wrist_radius}" length="${wrist_1_z if wrist_1_z > 0 else -wrist_1_z}" x="0" y="0" z="${wrist_1_visual_offset}" roll="0" pitch="0" yaw="0"/>
+      </xacro:if>
+      <xacro:if value="${collision_type == 'sphere'}">
+        <collision>
+          <origin xyz="0 0 ${wrist_1_visual_offset}" rpy="0 0 0"/>
+          <geometry>
+            <sphere radius="${wrist_radius}"/>
+          </geometry>
+        </collision>
+      </xacro:if>
+      <xacro:if value="${collision_type == 'box'}">
+        <collision>
+          <origin xyz="0 0 ${wrist_1_visual_offset}" rpy="0 0 0"/>
+          <geometry>
+            <box size="${2*wrist_radius} ${2*wrist_radius} ${wrist_1_z if wrist_1_z > 0 else -wrist_1_z}"/>
+          </geometry>
+        </collision>
+      </xacro:if>
       <inertial>
         <mass value="${wrist_1_mass}"/>
@@ -212,10 +363,40 @@
         </material>
       </visual>
-      <collision>
-        <origin xyz="0 0 ${wrist_2_visual_offset}" rpy="0 0 0"/>
-        <geometry>
-          <mesh filename="${wrist_2_collision_mesh}"/>
-        </geometry>
-      </collision>
+      <!-- Collision geometry: mesh or primitives based on collision_type -->
+      <xacro:if value="${collision_type == 'mesh'}">
+        <collision>
+          <origin xyz="0 0 ${wrist_2_visual_offset}" rpy="0 0 0"/>
+          <geometry>
+            <mesh filename="${wrist_2_collision_mesh}"/>
+          </geometry>
+        </collision>
+      </xacro:if>
+      <xacro:if value="${collision_type == 'cylinder'}">
+        <collision>
+          <origin xyz="0 0 ${wrist_2_visual_offset}" rpy="0 0 0"/>
+          <geometry>
+            <cylinder radius="${wrist_radius}" length="${wrist_2_y if wrist_2_y > 0 else -wrist_2_y}"/>
+          </geometry>
+        </collision>
+      </xacro:if>
+      <xacro:if value="${collision_type == 'capsule'}">
+        <xacro:capsule_collision radius="${wrist_radius}" length="${wrist_2_y if wrist_2_y > 0 else -wrist_2_y}" x="0" y="0" z="${wrist_2_visual_offset}" roll="0" pitch="0" yaw="0"/>
+      </xacro:if>
+      <xacro:if value="${collision_type == 'sphere'}">
+        <collision>
+          <origin xyz="0 0 ${wrist_2_visual_offset}" rpy="0 0 0"/>
+          <geometry>
+            <sphere radius="${wrist_radius}"/>
+          </geometry>
+        </collision>
+      </xacro:if>
+      <xacro:if value="${collision_type == 'box'}">
+        <collision>
+          <origin xyz="0 0 ${wrist_2_visual_offset}" rpy="0 0 0"/>
+          <geometry>
+            <box size="${2*wrist_radius} ${2*wrist_radius} ${wrist_2_y if wrist_2_y > 0 else -wrist_2_y}"/>
+          </geometry>
+        </collision>
+      </xacro:if>
       <inertial>
         <mass value="${wrist_2_mass}"/>
@@ -233,7 +414,17 @@
     <link name="${prefix}wrist_3_link">
       <xacro:property name="mesh_offset" value="${wrist_3_visual_offset_xyz}" scope="parent"/>
+      <xacro:property name="wrist_3_offset_x" value="0" scope="parent"/>
+      <xacro:property name="wrist_3_offset_y" value="0" scope="parent"/>
+      <xacro:property name="wrist_3_offset_z" value="${wrist_3_visual_offset}" scope="parent"/>
       <xacro:if value="${wrist_3_visual_offset_xyz == ''}">
         <xacro:property name="mesh_offset" value="0 0 ${wrist_3_visual_offset}" scope="parent"/>
       </xacro:if>
+      <xacro:unless value="${wrist_3_visual_offset_xyz == ''}">
+        <!-- Parse wrist_3_visual_offset_xyz string "x y z" into individual components -->
+        <xacro:property name="wrist_3_offset_parts" value="${wrist_3_visual_offset_xyz.split()}" scope="parent"/>
+        <xacro:property name="wrist_3_offset_x" value="${float(wrist_3_offset_parts[0])}" scope="parent"/>
+        <xacro:property name="wrist_3_offset_y" value="${float(wrist_3_offset_parts[1])}" scope="parent"/>
+        <xacro:property name="wrist_3_offset_z" value="${float(wrist_3_offset_parts[2])}" scope="parent"/>
+      </xacro:unless>
       <visual>
         <origin xyz="${mesh_offset}" rpy="${pi/2} 0 0"/>
@@ -245,10 +436,40 @@
         </material>
       </visual>
-      <collision>
-        <origin xyz="${mesh_offset}" rpy="${pi/2} 0 0"/>
-        <geometry>
-          <mesh filename="${wrist_3_collision_mesh}"/>
-        </geometry>
-      </collision>
+      <!-- Collision geometry: mesh or primitives based on collision_type -->
+      <xacro:if value="${collision_type == 'mesh'}">
+        <collision>
+          <origin xyz="${mesh_offset}" rpy="${pi/2} 0 0"/>
+          <geometry>
+            <mesh filename="${wrist_3_collision_mesh}"/>
+          </geometry>
+        </collision>
+      </xacro:if>
+      <xacro:if value="${collision_type == 'cylinder'}">
+        <collision>
+          <origin xyz="${mesh_offset}" rpy="0 0 0"/>
+          <geometry>
+            <cylinder radius="${wrist_radius}" length="${wrist_3_y if wrist_3_y > 0 else -wrist_3_y}"/>
+          </geometry>
+        </collision>
+      </xacro:if>
+      <xacro:if value="${collision_type == 'capsule'}">
+        <xacro:capsule_collision radius="${wrist_radius}" length="${wrist_3_y if wrist_3_y > 0 else -wrist_3_y}" x="${wrist_3_offset_x}" y="${wrist_3_offset_y}" z="${wrist_3_offset_z}" roll="0" pitch="0" yaw="0"/>
+      </xacro:if>
+      <xacro:if value="${collision_type == 'sphere'}">
+        <collision>
+          <origin xyz="${mesh_offset}" rpy="0 0 0"/>
+          <geometry>
+            <sphere radius="${wrist_radius}"/>
+          </geometry>
+        </collision>
+      </xacro:if>
+      <xacro:if value="${collision_type == 'box'}">
+        <collision>
+          <origin xyz="${mesh_offset}" rpy="0 0 0"/>
+          <geometry>
+            <box size="${2*wrist_radius} ${2*wrist_radius} ${wrist_3_y if wrist_3_y > 0 else -wrist_3_y}"/>
+          </geometry>
+        </collision>
+      </xacro:if>
       <inertial>
         <mass value="${wrist_3_mass}"/>

File: ur_description/urdf/ur.xacro (robot description, xacro)
@@ -17,4 +17,5 @@
    <xacro:arg name="safety_pos_margin" default="0.15"/>
    <xacro:arg name="safety_k_position" default="20"/>
+   <xacro:arg name="collision_type" default="mesh"/>
    <!-- arm -->
    <xacro:ur_robot
@@ -27,4 +28,5 @@
      safety_limits="$(arg safety_limits)"
      safety_pos_margin="$(arg safety_pos_margin)"
-     safety_k_position="$(arg safety_k_position)"/>
+     safety_k_position="$(arg safety_k_position)"
+     collision_type="$(arg collision_type)"/>
 </robot>

File: ur_description/urdf/ur10.xacro (robot description, xacro)
@@ -14,5 +14,6 @@
     Refer to 'inc/ur_macro.xacro' for more information.
   -->
+  <xacro:arg name="collision_type" default="mesh"/>
   <xacro:include filename="$(find ur_description)/urdf/inc/ur10_macro.xacro"/>
-  <xacro:ur10_robot prefix="" />
+  <xacro:ur10_robot prefix="" collision_type="$(arg collision_type)"/>
 </robot>

File: ur_description/urdf/ur10e.xacro (robot description, xacro)
@@ -14,5 +14,6 @@
     Refer to 'inc/ur_macro.xacro' for more information.
   -->
+  <xacro:arg name="collision_type" default="mesh"/>
   <xacro:include filename="$(find ur_description)/urdf/inc/ur10e_macro.xacro"/>
-  <xacro:ur10e_robot prefix="" />
+  <xacro:ur10e_robot prefix="" collision_type="$(arg collision_type)"/>
 </robot>

File: ur_description/urdf/ur12e.xacro (robot description, xacro)
@@ -14,5 +14,6 @@
     Refer to 'inc/ur_macro.xacro' for more information.
   -->
+  <xacro:arg name="collision_type" default="mesh"/>
   <xacro:include filename="$(find ur_description)/urdf/inc/ur12e_macro.xacro"/>
-  <xacro:ur12e_robot prefix="" />
+  <xacro:ur12e_robot prefix="" collision_type="$(arg collision_type)"/>
 </robot>
